File: hw/mini-usb-c-hub/aux-usb-c.kicad_sch (KiCad schematic)
At the start: 5 parts, among them J401 USB_C_Receptacle_USB2.0_16P

Commit message: chore(hw): update layout, fix references
Parts:
- renumbered C401 to C201, D401 to D201, J401 to J201, R402 to R201, R401 to R202
Connections:
- no-connect marks 0 -> 2
Changed lines of the file:
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@@
 		(color 0 0 0 0)
+	)
+	(no_connect
+		(at 132.08 85.09)
+	)
+	(no_connect
+		(at 132.08 87.63)
 	)
 	(wire
@@
 		(dnp no)
 		(fields_autoplaced yes)
-		(property "Reference" "R402"
+		(property "Reference" "R201"
 			(at 113.03 53.3399 0)
 			(effects
@@
 				)
 				(path "/7c04e056-0d84-4da3-ae50-c0eef25c6fa4/c0fa39e8-6859-419a-a123-dfe0bed56b96"
-					(reference "R402")
+					(reference "R301")
 					(unit 1)
 				)
@@
 		(on_board yes)
 		(dnp no)
-		(property "Reference" "D401"
+		(property "Reference" "D201"
 			(at 116.84 96.52 0)
 			(effects
@@
 			(project "mini-usb-c-hub"
 				(path "/7c04e056-0d84-4da3-ae50-c0eef25c6fa4/0cba7ead-2ce4-4d6f-80ca-d37204f10558"
-					(reference "D202")
+					(reference "D201")
 					(unit 1)
 				)
 				(path "/7c04e056-0d84-4da3-ae50-c0eef25c6fa4/c0fa39e8-6859-419a-a123-dfe0bed56b96"
-					(reference "D401")
+					(reference "D301")
 					(unit 1)
 				)
@@
 		(dnp no)
 		(fields_autoplaced yes)
-		(property "Reference" "#PWR0208"
+		(property "Reference" "#PWR0204"
 			(at 129.54 44.45 0)
 			(effects
@@
 			(project "mini-usb-c-hub"
 				(path "/7c04e056-0d84-4da3-ae50-c0eef25c6fa4/0cba7ead-2ce4-4d6f-80ca-d37204f10558"
-					(reference "#PWR0208")
+					(reference "#PWR0204")
 					(unit 1)
 				)
 				(path "/7c04e056-0d84-4da3-ae50-c0eef25c6fa4/c0fa39e8-6859-419a-a123-dfe0bed56b96"
-					(reference "#PWR0403")
+					(reference "#PWR0304")
 					(unit 1)
 				)
@@
 		(on_board yes)
 		(dnp no)
-		(property "Reference" "#PWR0405"
+		(property "Reference" "#PWR0203"
 			(at 120.65 44.45 0)
 			(effects
@@
 			(project "mini-usb-c-hub"
 				(path "/7c04e056-0d84-4da3-ae50-c0eef25c6fa4/0cba7ead-2ce4-4d6f-80ca-d37204f10558"
-					(reference "#PWR0207")
+					(reference "#PWR0203")
 					(unit 1)
 				)
 				(path "/7c04e056-0d84-4da3-ae50-c0eef25c6fa4/c0fa39e8-6859-419a-a123-dfe0bed56b96"
-					(reference "#PWR0405")
+					(reference "#PWR0303")
 					(unit 1)
 				)
@@
 		(dnp no)
 		(fields_autoplaced yes)
-		(property "Reference" "#PWR0404"
+		(property "Reference" "#PWR0202"
 			(at 105.41 107.95 0)
 			(effects
@@
 			(project "mini-usb-c-hub"
 				(path "/7c04e056-0d84-4da3-ae50-c0eef25c6fa4/0cba7ead-2ce4-4d6f-80ca-d37204f10558"
-					(reference "#PWR0206")
+					(reference "#PWR0202")
 					(unit 1)
 				)
 				(path "/7c04e056-0d84-4da3-ae50-c0eef25c6fa4/c0fa39e8-6859-419a-a123-dfe0bed56b96"
-					(reference "#PWR0404")
+					(reference "#PWR0302")
 					(unit 1)
 				)
@@
 		(dnp no)
 		(fields_autoplaced yes)
-		(property "Reference" "R401"
+		(property "Reference" "R202"
 			(at 123.19 53.3399 0)
 			(effects
@@
 				)
 				(path "/7c04e056-0d84-4da3-ae50-c0eef25c6fa4/c0fa39e8-6859-419a-a123-dfe0bed56b96"
-					(reference "R401")
+					(reference "R302")
 					(unit 1)
 				)
@@
 		(dnp no)
 		(fields_autoplaced yes)
-		(property "Reference" "#PWR0402"
+		(property "Reference" "#PWR0201"
 			(at 105.41 74.93 0)
 			(effects
@@
 			(project "mini-usb-c-hub"
 				(path "/7c04e056-0d84-4da3-ae50-c0eef25c6fa4/0cba7ead-2ce4-4d6f-80ca-d37204f10558"
-					(reference "#PWR0205")
+					(reference "#PWR0201")
 					(unit 1)
 				)
 				(path "/7c04e056-0d84-4da3-ae50-c0eef25c6fa4/c0fa39e8-6859-419a-a123-dfe0bed56b96"
-					(reference "#PWR0402")
+					(reference "#PWR0301")
 					(unit 1)
 				)
@@
 		(dnp no)
 		(fields_autoplaced yes)
-		(property "Reference" "C401"
+		(property "Reference" "C201"
 			(at 168.91 67.3099 0)
 			(effects
@@
 			(project "mini-usb-c-hub"
 				(path "/7c04e056-0d84-4da3-ae50-c0eef25c6fa4/0cba7ead-2ce4-4d6f-80ca-d37204f10558"
-					(reference "C202")
+					(reference "C201")
 					(unit 1)
 				)
 				(path "/7c04e056-0d84-4da3-ae50-c0eef25c6fa4/c0fa39e8-6859-419a-a123-dfe0bed56b96"
-					(reference "C401")
+					(reference "C301")
 					(unit 1)
 				)
@@
 		(on_board yes)
 		(dnp no)
-		(property "Reference" "J401"
+		(property "Reference" "J201"
 			(at 147.32 49.53 0)
 			(effects
@@
 			(project "mini-usb-c-hub"
 				(path "/7c04e056-0d84-4da3-ae50-c0eef25c6fa4/0cba7ead-2ce4-4d6f-80ca-d37204f10558"
-					(reference "J202")
+					(reference "J201")
 					(unit 1)
 				)
 				(path "/7c04e056-0d84-4da3-ae50-c0eef25c6fa4/c0fa39e8-6859-419a-a123-dfe0bed56b96"
-					(reference "J401")
+					(reference "J301")
 					(unit 1)
 				)
@@
 		(dnp no)
 		(fields_autoplaced yes)
-		(property "Reference" "#PWR0209"
+		(property "Reference" "#PWR0205"
 			(at 147.32 105.41 0)
 			(effects
@@
 			(project "mini-usb-c-hub"
 				(path "/7c04e056-0d84-4da3-ae50-c0eef25c6fa4/0cba7ead-2ce4-4d6f-80ca-d37204f10558"
-					(reference "#PWR0209")
+					(reference "#PWR0205")
 					(unit 1)
 				)
 				(path "/7c04e056-0d84-4da3-ae50-c0eef25c6fa4/c0fa39e8-6859-419a-a123-dfe0bed56b96"
-					(reference "#PWR0401")
-					(unit 1)
-				)
+					(reference "#PWR0305")
+					(unit 1)
+				)

Commit message: chore(hw): switch to KiCad 9.0
Changed lines of the file:
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@@
 (kicad_sch
-	(version 20231120)
+	(version 20250114)
 	(generator "eeschema")
-	(generator_version "8.0")
+	(generator_version "9.0")
 	(paper "A4")
 	(junction
@@
 		(shape bidirectional)
 		(at 83.82 74.93 180)
-		(fields_autoplaced yes)
 		(effects
 			(font
@@
 		(shape bidirectional)
 		(at 83.82 72.39 180)
-		(fields_autoplaced yes)
 		(effects
 			(font
